File: Borta Dators KiCad/Borta Dators.kicad_pcb (KiCad board)
At the start: 2 copper layers, 70 x 70 mm, 42 parts, among them J1 ST_LINK, J2 Micro_SD_Card, J3 Conn_02x12_Top_Bottom, J6 Bluetooth, Q1 BCX54, SW3 SW_Push

Commit message: Misc stuff update
Other:
- net class Default removed
